Commit message: update bot

File: ex05/robot_description/urdf/robot.urdf.xacro (robot description, xacro)
@@ -2,7 +2,6 @@
 <robot name="vacuum_robot" xmlns:xacro="http://ros.org/wiki/xacro">
     <xacro:include filename="$(find robot_description)/urdf/gazebo.urdf.xacro" />
-    <xacro:property name="chassis_length" value="0.4"/>
-    <xacro:property name="chassis_width" value="0.3"/>
-    <xacro:property name="chassis_height" value="0.1"/>
+    <xacro:property name="chassis_radius" value="0.2"/> <!-- Радиус корпуса -->
+    <xacro:property name="chassis_height" value="0.1"/> <!-- Высота корпуса -->
     <xacro:property name="wheel_radius" value="0.05"/>
     <xacro:property name="wheel_thickness" value="0.03"/>
@@ -15,5 +14,5 @@
     <xacro:property name="caster_wheel_offset_x" value="0.1"/>
     <xacro:property name="caster_wheel_offset_z" value="${wheel_offset_z - wheel_radius + caster_wheel_radius}"/>
-    <xacro:property name="mass" value="1.5"/>
+    <xacro:property name="mass" value="1.5"/> <!-- Масса корпуса -->
     <material name="white">
         <color rgba="1 1 1 1" />
@@ -37,27 +36,27 @@
         <parent link="base_link"/>
         <child link="chassis"/>
-        <origin xyz="${-wheel_offset_x} 0 ${-wheel_offset_z}"/>
+        <origin xyz="0 0 ${-wheel_offset_z}"/>
     </joint>
     <link name="chassis">
         <inertial>
-            <origin xyz="${chassis_length/2} 0 ${chassis_height/2}" rpy="0 0 0"/>
+            <origin xyz="0 0 ${chassis_height / 2}" rpy="0 0 0"/>
             <mass value="${mass}" />
-            <inertia ixx="${(1/12) * mass * (chassis_width*chassis_width + chassis_height*chassis_height)}"
+            <inertia ixx="${(1/2) * mass * (chassis_radius * chassis_radius)}"
                      ixy="0.0" ixz="0.0"
-                     iyy="${(1/12) * mass * (chassis_length*chassis_length + chassis_height*chassis_height)}"
+                     iyy="${(1/2) * mass * (chassis_radius * chassis_radius)}"
                      iyz="0.0"
-                     izz="${(1/12) * mass * (chassis_length*chassis_length + chassis_width*chassis_width)}" />
+                     izz="${(1/2) * mass * (chassis_radius * chassis_radius)}" />
         </inertial>
         <visual>
-            <origin xyz="${chassis_length/2} 0 ${chassis_height/2}"/>
+            <origin xyz="0 0 ${chassis_height / 2}"/>
             <geometry>
-                <box size="${chassis_length} ${chassis_width} ${chassis_height}"/>
+                <cylinder radius="${chassis_radius}" length="${chassis_height}"/> <!-- Цилиндр для корпуса -->
             </geometry>
             <material name="gray"/>
         </visual>
         <collision>
-            <origin xyz="${chassis_length/2} 0 ${chassis_height/2}"/>
+            <origin xyz="0 0 ${chassis_height / 2}"/>
             <geometry>
-                <box size="${chassis_length} ${chassis_width} ${chassis_height}"/>
+                <cylinder radius="${chassis_radius}" length="${chassis_height}"/> <!-- Цилиндр для коллизий -->
             </geometry>
         </collision>
